File: E&S_Datalogger/ES_Datalogger.sch (EAGLE design)
At the start: 17 parts, among them J1 CORTEX_DEBUG_PTH, U1 ATSAMD21G-A, U2 9DoF IMU, U4 MPL3115A2, Y1 32.768kHz

Commit message: Added board file
Parts:
- added C10, C11: 1uF, adafruit:C-USC0805
- added CN1: (no value), adafruit:JST_2PIN-SMT
- added CN3: (no value), adafruit:USBMOLEX
- added D2: (no value), adafruit:DIODE_SOD-123FL
- added JP1: (no value), pinhead:PINHD-1X4
- added JP2: (no value), pinhead:PINHD-1X5
- added LED1, LED2, LED3, LED4: (no value), adafruit:LEDCHIPLED_0805
- added R4, R5, R6, R7: 330, adafruit:R-US_R0805
- added U3: 3.3V, SparkFun-IC-Power:V_REG_AP2112K-3.3V
Connections:
- removed net N$8: U$1.CS
- new net GREEN_LED: LED3.A, U1.PB08(AIN2/SER4:0/TC4:0)
- new net N$3: LED1.C, R4.2
- new net N$5: LED2.C, R5.2
- new net N$6: LED3.C, R6.2
- new net N$7: LED4.C, R7.2
- new net RED_LED: LED4.A, U1.PB09(AIN3/SER4:1/TC4:1)
- new net RX_LED: LED1.A, U1.PB03(AIN11/SER5:1)
- new net SD_CS: U$1.CS, U1.PA08(I2C/AIN16/SER0:0+)
- new net TX_LED: LED2.A, U1.PA27
- new net VBUS: C10.1, CN3.VBUS, D2.C, U3.EN, U3.IN
- new net V_BAT: CN1.2, D2.A
- net GND: now also C10.2, C11.2, CN1.1, CN3.GND, JP1.1, JP2.1, R4.1, R5.1, R6.1, R7.1, U$1.VSS, U3.GND
- net MISO: now also JP2.4
- net MOSI: now also JP2.3
- net SCK: now also JP2.5
- net SCL: now also JP1.3
- net SDA: now also JP1.4
- net USB_D+: now also CN3.D+
- net USB_D-: now also CN3.D-
- net VDD: now also C11.1, JP1.2, JP2.2, U3.OUT
Other:
- moved on the sheet: C4, C6
