File: E&S_Datalogger/ES_Datalogger.sch (EAGLE design)
At the start: 36 parts, among them J1 CORTEX_DEBUG_PTH, U1 ATSAMD21G-A, U2 9DoF IMU, U3 3.3V, U4 MPL3115A2, Y1 32.768kHz

Commit message: Finished board and BoM
Parts:
- R4, R5, R6, R7: value 330 -> 100
- renumbered LED1 to RX, LED2 to TX, LED3 to STATUS, LED4 to ERROR
Changed lines of the file:
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@@
 <part name="U3" library="SparkFun-IC-Power" deviceset="V_REG_AP2112" device="K-3.3V" value="3.3V"/>
 <part name="JP1" library="pinhead" library_urn="urn:adsk.eagle:library:325" deviceset="PINHD-1X4" device="" package3d_urn="urn:adsk.eagle:package:22407/2"/>
-<part name="LED1" library="adafruit" deviceset="LED" device="CHIPLED_0805" value="Yellow"/>
-<part name="LED2" library="adafruit" deviceset="LED" device="CHIPLED_0805" value="Yellow"/>
-<part name="LED3" library="adafruit" deviceset="LED" device="CHIPLED_0805" value="Green"/>
-<part name="LED4" library="adafruit" deviceset="LED" device="CHIPLED_0805" value="Red"/>
-<part name="R4" library="adafruit" deviceset="R-US_" device="R0805" value="330"/>
-<part name="R5" library="adafruit" deviceset="R-US_" device="R0805" value="330"/>
-<part name="R6" library="adafruit" deviceset="R-US_" device="R0805" value="330"/>
-<part name="R7" library="adafruit" deviceset="R-US_" device="R0805" value="330"/>
+<part name="RX" library="adafruit" deviceset="LED" device="CHIPLED_0805" value="Yellow"/>
+<part name="TX" library="adafruit" deviceset="LED" device="CHIPLED_0805" value="Yellow"/>
+<part name="STATUS" library="adafruit" deviceset="LED" device="CHIPLED_0805" value="Green"/>
+<part name="ERROR" library="adafruit" deviceset="LED" device="CHIPLED_0805" value="Red"/>
+<part name="R4" library="adafruit" deviceset="R-US_" device="R0805" value="100"/>
+<part name="R5" library="adafruit" deviceset="R-US_" device="R0805" value="100"/>
+<part name="R6" library="adafruit" deviceset="R-US_" device="R0805" value="100"/>
+<part name="R7" library="adafruit" deviceset="R-US_" device="R0805" value="100"/>
 <part name="GND18" library="SparkFun-PowerSymbols" deviceset="GND" device=""/>
 <part name="S1" library="SparkFun-Switches" deviceset="MOMENTARY-SWITCH-SPST-2" device="-SMD-5.2MM"/>
@@
 <instance part="U3" gate="G$1" x="246.38" y="68.58"/>
 <instance part="JP1" gate="A" x="20.32" y="109.22" rot="R180"/>
-<instance part="LED1" gate="G$1" x="12.7" y="33.02"/>
-<instance part="LED2" gate="G$1" x="22.86" y="33.02"/>
-<instance part="LED3" gate="G$1" x="33.02" y="33.02"/>
-<instance part="LED4" gate="G$1" x="43.18" y="33.02"/>
+<instance part="RX" gate="G$1" x="12.7" y="33.02"/>
+<instance part="TX" gate="G$1" x="22.86" y="33.02"/>
+<instance part="STATUS" gate="G$1" x="33.02" y="33.02"/>
+<instance part="ERROR" gate="G$1" x="43.18" y="33.02"/>
 <instance part="R4" gate="G$1" x="12.7" y="20.32" rot="R90"/>
 <instance part="R5" gate="G$1" x="22.86" y="20.32" rot="R90"/>
@@
 </segment>
 <segment>
-<pinref part="LED1" gate="G$1" pin="A"/>
+<pinref part="RX" gate="G$1" pin="A"/>
 <wire x1="12.7" y1="35.56" x2="12.7" y2="38.1" width="0.1524" layer="91"/>
 <label x="12.7" y="38.1" size="1.27" layer="95" rot="R90" xref="yes"/>
@@
 </segment>
 <segment>
-<pinref part="LED2" gate="G$1" pin="A"/>
+<pinref part="TX" gate="G$1" pin="A"/>
 <wire x1="22.86" y1="35.56" x2="22.86" y2="38.1" width="0.1524" layer="91"/>
 <label x="22.86" y="38.1" size="1.27" layer="95" rot="R90" xref="yes"/>
@@
 </segment>
 <segment>
-<pinref part="LED3" gate="G$1" pin="A"/>
+<pinref part="STATUS" gate="G$1" pin="A"/>
 <wire x1="33.02" y1="35.56" x2="33.02" y2="38.1" width="0.1524" layer="91"/>
 <label x="33.02" y="38.1" size="1.27" layer="95" rot="R90" xref="yes"/>
@@
 </segment>
 <segment>
-<pinref part="LED4" gate="G$1" pin="A"/>
+<pinref part="ERROR" gate="G$1" pin="A"/>
 <wire x1="43.18" y1="35.56" x2="43.18" y2="38.1" width="0.1524" layer="91"/>
 <label x="43.18" y="38.1" size="1.27" layer="95" rot="R90" xref="yes"/>
@@
 <segment>
 <pinref part="R4" gate="G$1" pin="2"/>
-<pinref part="LED1" gate="G$1" pin="C"/>
+<pinref part="RX" gate="G$1" pin="C"/>
 <wire x1="12.7" y1="25.4" x2="12.7" y2="27.94" width="0.1524" layer="91"/>
 </segment>
@@
 <segment>
 <pinref part="R5" gate="G$1" pin="2"/>
-<pinref part="LED2" gate="G$1" pin="C"/>
+<pinref part="TX" gate="G$1" pin="C"/>
 <wire x1="22.86" y1="25.4" x2="22.86" y2="27.94" width="0.1524" layer="91"/>
 </segment>
@@
 <segment>
 <pinref part="R6" gate="G$1" pin="2"/>
-<pinref part="LED3" gate="G$1" pin="C"/>
+<pinref part="STATUS" gate="G$1" pin="C"/>
 <wire x1="33.02" y1="25.4" x2="33.02" y2="27.94" width="0.1524" layer="91"/>
 </segment>
@@
 <segment>
 <pinref part="R7" gate="G$1" pin="2"/>
-<pinref part="LED4" gate="G$1" pin="C"/>
+<pinref part="ERROR" gate="G$1" pin="C"/>
 <wire x1="43.18" y1="27.94" x2="43.18" y2="25.4" width="0.1524" layer="91"/>
 </segment>
