File: E&S_Datalogger/ES_Datalogger.brd (EAGLE design)
At the start: 35 x 45.7 mm, 36 parts, among them J1 CORTEX_DEBUG_PTH, U1 ATSAMD21G-A, U2 9DoF IMU, U3 3.3V, U4 MPL3115A2, Y1 32.768kHz

Commit message: Finished board and BoM
Parts:
- R4, R5, R6, R7: value 330 -> 100
- moved C8 0.51 mm to (6.35, 3.81)
- renumbered LED1 to RX, LED2 to TX, LED3 to STATUS, LED4 to ERROR
Routing:
- net GND: track 252.7 -> 253.3 mm
Other:
- board size 35 x 45.7 mm -> 35.5 x 45.7 mm
- board text added: "E&S DATALOGGER"
- board text added: "MISO"
- board text added: "MOSI"
- board text added: "RST"
- board text added: "SCK"
- board text added: "Vdd"
- board text removed: "E&S DATALOGGER R1"
